Commit message: change tool0 to iiwa_tool0 for dual arm setup

File: iiwa_description/urdf/iiwa.urdf.xacro (robot description, xacro)
@@ -169,5 +169,5 @@
       </inertial>
   </link>
-  <link name="${prefix}tool0"/>
+  <link name="${prefix}iiwa_tool0"/>
   <joint name="${prefix}joint_a1" type="revolute">
       <origin rpy="0 0 0" xyz="0 0 0"/>
@@ -222,5 +222,5 @@
       <origin rpy="0 0 0" xyz="0 0 0.154"/>
       <parent link="${prefix}link_7"/>
-      <child link="${prefix}tool0"/>
+      <child link="${prefix}iiwa_tool0"/>
       <axis xyz="0 0 0"/>
   </joint>
